Commit message: added laser to urdf

File: raw_description/urdf/base_short/base.urdf.xacro (robot description, xacro)
@@ -5,4 +5,5 @@
   <!-- drive_wheel module -->
   <xacro:include filename="$(find cob_description)/urdf/drive_wheel/drive_wheel.urdf.xacro" />
+  <xacro:include filename="$(find cob_description)/urdf/sensors/sick_s300_laser.urdf.xacro"/>
   <!-- properties -->
   <xacro:property name="caster_offset_x" value="0.228" />  <!--modify here-->
@@ -97,4 +98,12 @@
       <origin xyz="${-battery_offset_x} ${battery_offset_y} ${battery_offset_z}" rpy="${M_PI/2} 0 ${-M_PI/2}" />
     </xacro:cob_batteries>
+    <!-- base laser front -->
+    <xacro:sick_s300_laser_v0 name="${name}_laser_front" parent="${name}">
+      <origin xyz="${laser_front_x} ${laser_front_y} ${laser_front_z}" rpy="${laser_front_roll} ${laser_front_pitch} ${laser_front_yaw}" />
+    </xacro:sick_s300_laser_v0>
+    <!-- base laser rear -->
+    <xacro:sick_s300_laser_v0 name="${name}_laser_rear" parent="${name}">
+      <origin xyz="${laser_rear_x} ${laser_rear_y} ${laser_rear_z}" rpy="${laser_rear_roll} ${laser_rear_pitch} ${laser_rear_yaw}" />
+    </xacro:sick_s300_laser_v0>
     <!-- gazebo extensions -->
     <xacro:base_gazebo name="${name}" />
