Commit message: Remove fixed stuff from description

File: cob_description/urdf/robotrainer2/base.urdf.xacro (robot description, xacro)
@@ -8,10 +8,7 @@
   <xacro:property name="telescope_rot_angle_min" value="16" />
   <xacro:property name="telescope_rot_angle_max" value="36" />
-<!--  <xacro:property name="telescope_rot_angle" value="16" />
-  <xacro:property name="telescope_rot_rad" value="${M_PI*telescope_rot_angle/180}" />-->
   <!-- linear values from 0.274 to 0.474 with the step of 5 cm -->
   <xacro:property name="telescope_linear_pos_min" value="0.274" />
   <xacro:property name="telescope_linear_pos_max" value="0.424" />
-<!--   <xacro:property name="telescope_linear_pos" value="0.274" /> -->
   <xacro:property name="caster_offset_back_x" value="0.210992" />  <!--modify here-->
   <xacro:property name="caster_offset_back_y" value="0.0" />

Commit message: Remove telescope fixed transformation

File: cob_description/urdf/robotrainer2/base.urdf.xacro (robot description, xacro)
@@ -119,10 +119,4 @@
       </collision>-->
     </link>
-<!--    <joint name="${name}_bl_chassis_bl_telescope_lin_joint" type="fixed">
-      <origin xyz="${telescope_linear_pos} 0 0" rpy="0 0 0" />
-      <parent link="${name}_baseplate_bl_telescope_rot_link"/>
-      <child link="${name}_baseplate_bl_telescope_lin_link" />
-    </joint>
-    -->
     <joint name="${name}_bl_chassis_bl_telescope_lin_joint" type="prismatic">
       <origin xyz="0 0 0" rpy="0 0 0" />
@@ -132,9 +126,4 @@
       <child link="${name}_baseplate_bl_telescope_lin_link" />
     </joint>
-<!--    <joint name="${name}_br_chassis_br_telescope_lin_joint" type="fixed">
-      <origin xyz="${telescope_linear_pos} 0 0" rpy="0 0 0" />
-      <parent link="${name}_baseplate_br_telescope_rot_link"/>
-      <child link="${name}_baseplate_br_telescope_lin_link" />
-    </joint>-->
     <joint name="${name}_br_chassis_br_telescope_lin_joint" type="prismatic">
       <origin xyz="0 0 0" rpy="0 0 0" />
